File: TritLed/TritLed.kicad_pcb (KiCad board)
At the start: 2 copper layers, 39.4 x 27.9 mm, 9 parts, among them P1 Power&In, U1 LM393

Commit message: Изображения
Signed-off-by: Алексей Кляузер <drum@pisem.net>
Parts:
- moved R2 2.54 mm to (52.1, 39.4)
- moved R3 1.27 mm to (48.3, 39.4)
- moved R4 1.27 mm to (33.0, 36.8)
Routing:
- net Net-(P1-Pad3): track 25.4 -> 30.5 mm
- net Net-(R2-Pad2): track 7.62 -> 10.2 mm
- net Net-(R1-Pad2): track 27.9 -> 30.5 mm
- net Net-(R4-Pad2): track 5.08 -> 6.35 mm
- net Net-(D1-Pad2): track 5.08 -> 3.81 mm
Other:
- board text added: "+"
- board text added: "+2,5В"
- board text added: "-"
- board text added: "-2,5В"
